Commit message: Adding dummy point cloud

File: robot/ros_ws/src/base_moveit_config_2/config/demo_bot.ros2_control.xacro (robot description, xacro)
@@ -64,4 +64,44 @@
                 <state_interface name="velocity"/>
             </joint>
+            <joint name="Revolute_1">
+                <state_interface name="position">
+                    <param name="initial_value">0.0</param>
+                </state_interface>
+            </joint>
+            <joint name="Revolute_2">
+                <state_interface name="position">
+                    <param name="initial_value">0.0</param>
+                </state_interface>
+            </joint>
+            <joint name="Revolute_3">
+                <state_interface name="position">
+                    <param name="initial_value">0.0</param>
+                </state_interface>
+            </joint>
+            <joint name="Revolute_4">
+                <state_interface name="position">
+                    <param name="initial_value">0.0</param>
+                </state_interface>
+            </joint>
+            <joint name="Revolute_5">
+                <state_interface name="position">
+                    <param name="initial_value">0.0</param>
+                </state_interface>
+            </joint>
+            <joint name="Revolute_6">
+                <state_interface name="position">
+                    <param name="initial_value">0.0</param>
+                </state_interface>
+            </joint>
+            <joint name="Revolute_7">
+                <state_interface name="position">
+                    <param name="initial_value">0.0</param>
+                </state_interface>
+            </joint>
+            <joint name="Revolute_8">
+                <state_interface name="position">
+                    <param name="initial_value">0.0</param>
+                </state_interface>
+            </joint>
         </ros2_control>
     </xacro:macro>

Commit message: Basic moveit+IsaacSim setup

File: robot/ros_ws/src/base_moveit_config_2/config/demo_bot.ros2_control.xacro (robot description, xacro)
@@ -6,5 +6,8 @@
             <hardware>
                 <!-- By default, set up controllers for simulation. This won't work on real hardware -->
-                <plugin>mock_components/GenericSystem</plugin>
+                <!-- <plugin>mock_components/GenericSystem</plugin> -->
+                <plugin>topic_based_ros2_control/TopicBasedSystem</plugin>
+                <param name="joint_commands_topic">/isaac/joint_commands</param>
+                <param name="joint_states_topic">/isaac/joint_states</param>
             </hardware>
             <joint name="Revolute_9">
@@ -64,44 +67,44 @@
                 <state_interface name="velocity"/>
             </joint>
-            <joint name="Revolute_1">
-                <state_interface name="position">
+            <!-- <joint name="Revolute_1">
+                <command_interface name="position"/> <state_interface name="position">
                     <param name="initial_value">0.0</param>
                 </state_interface>
             </joint>
             <joint name="Revolute_2">
-                <state_interface name="position">
+                <command_interface name="position"/> <state_interface name="position">
                     <param name="initial_value">0.0</param>
                 </state_interface>
             </joint>
             <joint name="Revolute_3">
-                <state_interface name="position">
+                <command_interface name="position"/><state_interface name="position">
                     <param name="initial_value">0.0</param>
                 </state_interface>
             </joint>
             <joint name="Revolute_4">
-                <state_interface name="position">
+                <command_interface name="position"/> <state_interface name="position">
                     <param name="initial_value">0.0</param>
                 </state_interface>
             </joint>
             <joint name="Revolute_5">
-                <state_interface name="position">
+                <command_interface name="position"/> <state_interface name="position">
                     <param name="initial_value">0.0</param>
                 </state_interface>
             </joint>
             <joint name="Revolute_6">
-                <state_interface name="position">
+                <command_interface name="position"/> <state_interface name="position">
                     <param name="initial_value">0.0</param>
                 </state_interface>
             </joint>
             <joint name="Revolute_7">
-                <state_interface name="position">
+                <command_interface name="position"/> <state_interface name="position">
                     <param name="initial_value">0.0</param>
                 </state_interface>
             </joint>
             <joint name="Revolute_8">
-                <state_interface name="position">
+                <command_interface name="position"/> <state_interface name="position">
                     <param name="initial_value">0.0</param>
                 </state_interface>
-            </joint>
+            </joint>             -->
         </ros2_control>
     </xacro:macro>
