Commit message: commit local planning changes from SVD

File: robot/ros_ws/src/autonomy/5_planning/base_urdf/robot.urdf (robot description, URDF)
Before this commit: robot demo_bot, 20 links, 19 joints
Links:
- added link base_top_link; collision box size=0.01410 0.12771 0.08543
- added link cube_angle_link; collision box size=0.05 1 0.5
- added link cube_link; collision box size=0.05 1 0.5
- added link wellplate_link; collision box size=0.12771 0.01410 0.08543
- link Finger_left_2: geometry collision mesh filename=package://base_urdf/meshes/Finger_left_2.stl scale=1 1.5 1; visual mesh filename=package://base_urdf/meshes/Finger_left_2.stl
- link Finger_right_2: geometry collision mesh filename=package://base_urdf/meshes/Finger_right_2.stl scale=1 1.5 1; visual mesh filename=package://base_urdf/meshes/Finger_right_2.stl
Joints:
- added joint base_top_joint: type fixed, parent Chassis_1, child base_top_link, origin xyz=-0.1 0.0 0.078 rpy=0.0 0.0 0.0
- added joint cube_angle_joint: type fixed, parent Chassis_1, child cube_angle_link, origin xyz=0.05 0.0 -0.65 rpy=0.0 0.523598776 0.0
- added joint cube_joint: type fixed, parent Chassis_1, child cube_link, origin xyz=0.16 0.2 -0.15 rpy=0.0 0.0 0.0
- added joint wellplate_joint: type fixed, parent Finger_left_2, child wellplate_link, origin xyz=0 0.08 0.075 rpy=0.0 0.0 0.0
- joint Slider_1: origin xyz=0.0161 0.0007 -0.06 rpy=-1.5707963 0 1.623 -> xyz=0.066 0.0007 -0.06 rpy=-1.5707963 0 1.623
- joint Slider_2: origin xyz=-0.0186 -0.001 -0.06 rpy=1.5707963 0 1.623 -> xyz=-0.066 -0.001 -0.06 rpy=1.5707963 0 1.623

Commit message: prm implemented with jagged paths

File: robot/ros_ws/src/autonomy/5_planning/base_urdf/robot.urdf (robot description, URDF)
Before this commit: robot demo_bot, 24 links, 23 joints
Links:
- added link wellplate_holder_link; collision box size=0.32 0.65 0.025
- link cube_angle_link: geometry collision box size=0.05 0.35 0.8
- link cube_link: geometry collision box size=0.025 0.35 0.5
- link wellplate_link: geometry collision box size=0.004 0.01410 0.08543
Joints:
- added joint wellplate_holder_joint: type fixed, parent Chassis_1, child wellplate_holder_link, origin xyz=0 +0.2 0.14 rpy=0.0 0 0.0
- joint cube_angle_joint: origin xyz=0.05 0.0 -0.65 rpy=0.0 0.523598776 0.0 -> xyz=0.05 0.2 -0.65 rpy=0.0 0.523598776 0.0
