Commit message: Add gripper side clearance box; update planning run docs
- robot.urdf: extra 4 cm collision slab on the -x side of gripper_v43_1
  (from local_changes 3d98a7e), so plans keep sideways clearance.
- Planning ReadMe and docs/launch-planning.md: run with the camera hub on
  the Xavier and camera_perception on the Thor instead of pc3.py; note
  that the obstacle cloud is frozen at the first plan command.
- calibrate-top-camera.md, launch-visual-servo.md: renumbered step links.

Co-Authored-By: Claude Opus 5.5 <noreply@anthropic.com>

File: robot/ros_ws/src/autonomy/5_planning/base_urdf/robot.urdf (robot description, URDF)
Before this commit: robot demo_bot, 25 links, 24 joints
Links:
- link gripper_v43_1: geometry collision box size=0.04 0.075 0.0745; collision mesh filename=package://base_urdf/meshes/gripper_v43_1.stl
