Commit message: local changes on Thor

File: robot/ros_ws/src/autonomy/5_planning/base_urdf/robot.urdf (robot description, URDF)
Before this commit: robot demo_bot, 25 links, 24 joints
Links:
- link gripper_v43_1: geometry collision box size=0.10 0.075 0.0745; collision mesh filename=package://base_urdf/meshes/gripper_v43_1.stl
