Commit message: New Sim

File: robot/ros_ws/src/autonomy/5_planning/base_urdf/robot_isaac.urdf (robot description, URDF)
Before this commit: robot demo_bot, 18 links, 17 joints
Links:
- added link base_footprint
- added link zed_x_left_camera
- added link zed_x_mount
- added link zed_x_nano_left_camera
- added link zed_x_nano_mount
Joints:
- added joint base_footprint_to_chassis: type fixed, parent base_footprint, child Chassis_1, origin xyz=0 0 0.89259868 rpy=3.141592653589793 0 0
- added joint zed_x_left_optical_joint: type fixed, parent zed_x_mount, child zed_x_left_camera, origin xyz=0 0 0 rpy=-1.570796326794897 -1.570796326794897 -1.570796326794897
- added joint zed_x_mount_joint: type fixed, parent base_footprint, child zed_x_mount, origin xyz=0.08318796 0.03996821 1.50901977 rpy=-0.00002608 0.52735827 -0.00600658
- added joint zed_x_nano_left_optical_joint: type fixed, parent zed_x_nano_mount, child zed_x_nano_left_camera, origin xyz=0 0 0 rpy=-1.570796326794897 0 -1.570796326794897
- added joint zed_x_nano_mount_joint: type fixed, parent gripper_v43_1, child zed_x_nano_mount, origin xyz=0.05207864 0.03019945 -0.04880624 rpy=-1.51883872 0.05957537 -1.70751561
